File: schematic/WirelessDS18B20.sch (KiCad schematic (older format))
At the start: 14 parts, among them P1 Power Connector, P2 1-Wire Bus, P3 SERIAL_TX, Q1 BS170, SW1 SW_Push, SW2 SW_Push, U1 AMS1117-3.3, U2 ESP-01

Commit message: Switch schematic to D1 Mini
Parts:
- removed C1: 10uF, Capacitors_Tantalum_SMD:CP_Tantalum_Case-A_EIA-3216-18_Hand, symbol CP
- removed C2: 100uF, Capacitors_Tantalum_SMD:CP_Tantalum_Case-B_EIA-3528-21_Hand, symbol CP
- removed D1: SS34, Diodes_SMD_Custom:SMA_Handsoldering_Custom, symbol D_Schottky
- removed P1: Power Connector, Connect:bornier2, symbol Conn_01x02
- removed P3: SERIAL_TX, Pin_Headers:Pin_Header_Straight_1x02, symbol Conn_01x02
- removed SW1, SW2: SW_Push, Buttons_Switches_ThroughHole:SW_PUSH_6mm, symbol SW_Push
- removed U1: AMS1117-3.3, TO_SOT_Packages_SMD:SOT-223, symbol LM1117-3.3
- removed U2: ESP-01, ESP8266:ESP-01, symbol ESP-01v090
- added U1: WeMos_mini, wemos_d1_mini:wemos-d1-mini-DIL-only, symbol wemos_mini:WeMos_mini
- P2: footprint Connect:bornier3 -> Terminal_Blocks:TerminalBlock_bornier-3_P5.08mm; symbol Conn_01x03 -> Connector_Generic:Conn_01x03
- Q1: footprint TO_SOT_Packages_THT:TO-92_Molded_Narrow_Oval -> TO_SOT_Packages_THT:TO-92_Horizontal2_Inline_Narrow_Oval; symbol BS170 -> Transistor_FET:BS170
- R1, R2, R3: symbol R -> Device:R
Connections:
- wire segments 46 -> 24
- no-connect marks 0 -> 12
Other:
- note added: "V2.1"
- moved on the sheet: Q1
