File: schematic/WirelessDS18B20.kicad_pcb (KiCad board)
At the start: 2 copper layers, 25.4 x 33.7 mm, 8 parts, among them P1 1-Wire Bus, Q1 MMBF170, U1 WeMos_mini, U2 AMS1117-3.3

Commit message: Update of schematic
Parts:
- Q1: value MMBF170 -> 2N7002
Changed lines of the file:
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@@
 	(setup
 		(pad_to_mask_clearance 0)
-		(solder_mask_min_width 0.25)
 		(allow_soldermask_bridges_in_footprints no)
 		(pcbplotparams
@@
 			(plot_on_all_layers_selection 0x0000000_00000000)
 			(disableapertmacros no)
-			(usegerberextensions no)
+			(usegerberextensions yes)
 			(usegerberattributes no)
 			(usegerberadvancedattributes no)
@@
 			(plotinvisibletext no)
 			(sketchpadsonfab no)
-			(subtractmaskfromsilk no)
+			(subtractmaskfromsilk yes)
 			(outputformat 1)
 			(mirror no)
@@
 			)
 		)
+		(property "LCSC" "C119052"
+			(at 0 0 90)
+			(unlocked yes)
+			(layer "F.Fab")
+			(hide yes)
+			(effects
+				(font
+					(size 1 1)
+					(thickness 0.15)
+				)
+			)
+		)
 		(property ki_fp_filters "CP_*")
 		(sheetname "Root")
@@
 		(tags "capacitor tantalum")
 		(property "Reference" "C2"
-			(at 1.66 2.159 360)
+			(at 1.66 2.159 0)
 			(layer "F.SilkS")
 			(effects
@@
 		)
 		(property "Value" "100u"
-			(at -1.769 2.159 360)
+			(at -1.769 2.159 0)
 			(layer "F.SilkS")
 			(effects
@@
 		)
 		(property "Footprint" "Capacitor_Tantalum_SMD:CP_EIA-3528-21_Kemet-B_Pad1.50x2.35mm_HandSolder"
-			(at 0 0 360)
+			(at 0 0 0)
 			(layer "B.Fab")
 			(hide yes)
@@
 		)
 		(property "Datasheet" ""
-			(at 0 0 360)
+			(at 0 0 0)
 			(layer "B.Fab")
 			(hide yes)
@@
 		)
 		(property "Description" "Polarized capacitor"
-			(at 0 0 360)
+			(at 0 0 0)
 			(layer "B.Fab")
 			(hide yes)
@@
 				)
 				(justify mirror)
+			)
+		)
+		(property "LCSC" "C129289"
+			(at 0 0 180)
+			(unlocked yes)
+			(layer "F.Fab")
+			(hide yes)
+			(effects
+				(font
+					(size 1 1)
+					(thickness 0.15)
+				)
 			)
 		)
@@
 		)
 		(fp_text user "${REFERENCE}"
-			(at 0 0 360)
+			(at 0 0 0)
 			(layer "F.Fab")
 			(effects
@@
 		(sheetname "Root")
 		(sheetfile "WirelessDS18B20.kicad_sch")
-		(attr through_hole)
+		(attr through_hole exclude_from_pos_files exclude_from_bom)
 		(fp_line
 			(start -2.54 -3.81)
@@
 		(tags "resistor handsolder")
 		(property "Reference" "R1"
-			(at 0 -1.65 360)
+			(at 0 -1.65 0)
 			(layer "F.SilkS")
 			(effects
@@
 		)
 		(property "Value" "1K"
-			(at 0 1.65 360)
+			(at 0 1.65 0)
 			(layer "F.SilkS")
 			(effects
@@
 				(font
 					(size 1.27 1.27)
+					(thickness 0.15)
+				)
+			)
+		)
+		(property "LCSC" "C17513"
+			(at 0 0 180)
+			(unlocked yes)
+			(layer "F.Fab")
+			(hide yes)
+			(effects
+				(font
+					(size 1 1)
 					(thickness 0.15)
 				)
@@
 		)
 		(fp_text user "${REFERENCE}"
-			(at 0 0 360)
+			(at 0 0 0)
 			(layer "F.Fab")
 			(effects
@@
 		(tags "resistor handsolder")
 		(property "Reference" "R3"
-			(at 0 -1.65 360)
+			(at 0 -1.65 0)
 			(layer "F.SilkS")
 			(effects
@@
 		)
 		(property "Value" "2.2K"
-			(at 0 1.65 360)
+			(at 0 1.65 0)
 			(layer "F.SilkS")
 			(effects
@@
 				(font
 					(size 1.27 1.27)
+					(thickness 0.15)
+				)
+			)
+		)
+		(property "LCSC" "C17520"
+			(at 0 0 180)
+			(unlocked yes)
+			(layer "F.Fab")
+			(hide yes)
+			(effects
+				(font
+					(size 1 1)
 					(thickness 0.15)
 				)
@@
 		)
 		(fp_text user "${REFERENCE}"
-			(at 0 0 360)
+			(at 0 0 0)
 			(layer "F.Fab")
 			(effects
@@
 			)
 		)
+		(property "LCSC" "C6186"
+			(at 0 0 90)
+			(unlocked yes)
+			(layer "F.Fab")
+			(hide yes)
+			(effects
+				(font
+					(size 1 1)
+					(thickness 0.15)
+				)
+			)
+		)
 		(property ki_fp_filters "SOT?223*TabPin2*")
 		(sheetname "Root")
@@
 		)
 		(fp_text user "${REFERENCE}"
-			(at 0 0 360)
+			(at 0 0 0)
 			(layer "F.Fab")
 			(effects
@@
 	)
 	(footprint "Package_TO_SOT_SMD:SOT-23_Handsoldering"
-		(placed yes)
 		(layer "F.Cu")
 		(at 32.07 38.505 90)
@@
 		(tags "SOT-23")
 		(property "Reference" "Q1"
-			(at 0 2.45 90)
-			(layer "F.SilkS")
-			(effects
-				(font
-					(size 1 1)
-					(thickness 0.15)
-				)
-			)
-		)
-		(property "Value" "MMBF170"
-			(at -0.23 -2.7 90)
+			(at 0 2.855 90)
+			(layer "F.SilkS")
+			(effects
+				(font
+					(size 1 1)
+					(thickness 0.15)
+				)
+			)
+		)
+		(property "Value" "2N7002"
+			(at 0 -2.86 90)
 			(layer "F.SilkS")
 			(effects
@@
 			)
 		)
-		(property "Datasheet" "https://www.diodes.com/assets/Datasheets/ds30104.pdf"
+		(property "Datasheet" "https://www.onsemi.com/pub/Collateral/NDS7002A-D.PDF"
 			(at 0 0 90)
 			(unlocked yes)
@@
 			)
 		)
-		(property "Description" "0.5A Id, 60V Vds, N-Channel MOSFET, SOT-23"
+		(property "Description" "0.115A Id, 60V Vds, N-Channel MOSFET, SOT-23"
 			(at 0 0 90)
 			(unlocked yes)
@@
 				(font
 					(size 1.27 1.27)
+					(thickness 0.15)
+				)
+			)
+		)
+		(property "LCSC" "C8545"
+			(at 0 0 90)
+			(unlocked yes)
+			(layer "F.Fab")
+			(hide yes)
+			(effects
+				(font
+					(size 1 1)
 					(thickness 0.15)
 				)
@@
 		(sheetname "Root")
 		(sheetfile "WirelessDS18B20.kicad_sch")
-		(attr through_hole)
+		(attr through_hole exclude_from_pos_files exclude_from_bom)
 		(fp_line
 			(start -18.46 -13.5)

Commit message: Update schematic
Parts:
- added Q2: 2N7002, Package_TO_SOT_SMD:SOT-23_Handsoldering, F.Cu at (29.7, 37.6)
- R2: renamed from R3; value 2.2K -> 3.3K
- moved C2 10.2 mm to (30.2, 42.7)
- moved R2 9.82 mm to (42.4, 38.9)
- moved U2 7.31 mm to (39.6, 44.2), turned to 0 degrees
- moved Q1 3.85 mm to (35.8, 37.6), turned to 180 degrees
- moved C1 1.78 mm to (31.0, 46.5), turned to 180 degrees
- moved R1 1.44 mm to (42.4, 36.3)
Connections:
- Q1 pad 3: Net-(P1-Pin_2) -> Net-(Q1-D)
- R2 pad 1: Net-(U1-D6) -> VCC
- R2 pad 2: Net-(Q1-G) -> Net-(Q1-D)
- U1 pad 13: Net-(U1-D6) -> Net-(Q1-G)
Routing:
- net Net-(Q1-G): track 4.56 -> 35.7 mm
- net Net-(U1-D6): track 13.5 -> 0.00 mm, vias 1 -> 0
- net Net-(Q1-D): track 0.00 -> 12.6 mm
- net GND: track 43.3 -> 54.4 mm
- net 5V: track 22.2 -> 13.0 mm
- net Net-(P1-Pin_2): track 43.1 -> 44.1 mm
- net VCC: track 27.2 -> 28.2 mm
Other:
- board size 25.4 x 33.7 mm -> 25.4 x 26.3 mm
- board text added: "Domochip WDS18B20"
- board text added: "R1: 1K R2: 3.3K Q1,Q2: 2N7002 C1: 10u C2: 100u U2: AMS1117-3.3"
- board text added: "V3.1"
- board text removed: "DomoChip WDS18B20 V3.0"
