File: schematic/WDS18B20.kicad_sch (KiCad schematic)
At the start: 10 parts, among them J1 WeMos_mini_Hat_Left, J2 WeMos_mini_Hat_Right, J3 1-Wire Bus, Q1 2N7002, Q2 2N7002, U2 AMS1117-3.3

Commit message: Update schematic
Parts:
- C1, C2, J3: JlcRotOffset (none) -> 180
Changed lines of the file:
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@@
+			)
+		)
+		(property "JlcRotOffset" "180"
+			(at 22.86 68.58 0)
+			(effects
+				(font
+					(size 1.27 1.27)
+				)
+				(hide yes)
 			)
 		)
@@
 		)
 		(property "LCSC" "C16133"
+			(at 44.45 68.58 0)
+			(effects
+				(font
+					(size 1.27 1.27)
+				)
+				(hide yes)
+			)
+		)
+		(property "JlcRotOffset" "180"
 			(at 44.45 68.58 0)
 			(effects
@@
 			(at 85.09 34.29 0)
 			(effects
+				(font
+					(size 1.27 1.27)
+				)
+				(hide yes)
+			)
+		)
+		(property "JlcRotOffset" "180"
+			(at 85.09 34.29 0)
+			(effects
